File: nRF52832.sch (KiCad schematic (older format))
At the start: 18 parts, among them U1 nRF52832-QFAA, X1 32MHz, X2 32.768kHz

Commit message: PCB Design
Parts:
- C1, C11, C12, C2, C3, C4, C5, C6, C7, C8: footprint (none) -> Capacitor_SMD:C_0402_1005Metric
- C10, C9: footprint (none) -> Capacitor_SMD:C_0603_1608Metric
- L1, L3: footprint (none) -> Inductor_SMD:L_0402_1005Metric
- L2: footprint (none) -> Inductor_SMD:L_0603_1608Metric
- U1: footprint (none) -> Package_DFN_QFN:QFN-48-1EP_6x6mm_P0.4mm_EP4.2x4.2mm
- X1: footprint (none) -> Crystal:Crystal_SMD_2016-4Pin_2.0x1.6mm
- X2: footprint (none) -> Crystal:Crystal_SMD_3215-2Pin_3.2x1.5mm
Changed lines of the file:
@@
 EESchema Schematic File Version 4
+LIBS:nRF52832-cache
 EELAYER 29 0
 EELAYER END
@@
 F 0 "C1" V 9000 2700 50  0000 C CNN
 F 1 "12pF" V 9300 2700 50  0000 C CNN
-F 2 "" H 9188 2550 50  0001 C CNN
+F 2 "Capacitor_SMD:C_0402_1005Metric" H 9188 2550 50  0001 C CNN
 F 3 "~" H 9150 2700 50  0001 C CNN
 	1    9150 2700
@@
 F 0 "C3" H 8415 4096 50  0000 L CNN
 F 1 "0.8pF" H 8415 4005 50  0000 L CNN
-F 2 "" H 8338 3900 50  0001 C CNN
+F 2 "Capacitor_SMD:C_0402_1005Metric" H 8338 3900 50  0001 C CNN
 F 3 "~" H 8300 4050 50  0001 C CNN
 	1    8300 4050
@@
 F 0 "C9" H 4115 2596 50  0000 L CNN
 F 1 "4.7µF" H 4115 2505 50  0000 L CNN
-F 2 "" H 4038 2400 50  0001 C CNN
+F 2 "Capacitor_SMD:C_0603_1608Metric" H 4038 2400 50  0001 C CNN
 F 3 "~" H 4000 2550 50  0001 C CNN
 	1    4000 2550
@@
 F 0 "C7" V 9000 3150 50  0000 C CNN
 F 1 "100pF" V 9300 3150 50  0000 C CNN
-F 2 "" H 9188 3000 50  0001 C CNN
+F 2 "Capacitor_SMD:C_0402_1005Metric" H 9188 3000 50  0001 C CNN
 F 3 "~" H 9150 3150 50  0001 C CNN
 	1    9150 3150
@@
 F 0 "C6" V 9000 3550 50  0000 C CNN
 F 1 "NC" V 9300 3550 50  0000 C CNN
-F 2 "" H 9188 3400 50  0001 C CNN
+F 2 "Capacitor_SMD:C_0402_1005Metric" H 9188 3400 50  0001 C CNN
 F 3 "~" H 9150 3550 50  0001 C CNN
 	1    9150 3550
@@
 F 0 "C10" H 5965 1496 50  0000 L CNN
 F 1 "1.0µF" H 5965 1405 50  0000 L CNN
-F 2 "" H 5888 1300 50  0001 C CNN
+F 2 "Capacitor_SMD:C_0603_1608Metric" H 5888 1300 50  0001 C CNN
 F 3 "~" H 5850 1450 50  0001 C CNN
 	1    5850 1450
@@
 F 0 "C2" V 9000 2200 50  0000 C CNN
 F 1 "12pF" V 9300 2200 50  0000 C CNN
-F 2 "" H 9188 2050 50  0001 C CNN
+F 2 "Capacitor_SMD:C_0402_1005Metric" H 9188 2050 50  0001 C CNN
 F 3 "~" H 9150 2200 50  0001 C CNN
 	1    9150 2200
@@
 F 0 "C4" H 3415 2596 50  0000 L CNN
 F 1 "100nF" H 3415 2505 50  0000 L CNN
-F 2 "" H 3338 2400 50  0001 C CNN
+F 2 "Capacitor_SMD:C_0402_1005Metric" H 3338 2400 50  0001 C CNN
 F 3 "~" H 3300 2550 50  0001 C CNN
 	1    3300 2550
@@
 F 0 "C5" H 4665 5496 50  0000 L CNN
 F 1 "100nF" H 4665 5405 50  0000 L CNN
-F 2 "" H 4588 5300 50  0001 C CNN
+F 2 "Capacitor_SMD:C_0402_1005Metric" H 4588 5300 50  0001 C CNN
 F 3 "~" H 4550 5450 50  0001 C CNN
 	1    4550 5450
@@
 F 0 "C11" V 2000 3150 50  0000 C CNN
 F 1 "12pF" V 2300 3150 50  0000 C CNN
-F 2 "" H 2188 3000 50  0001 C CNN
+F 2 "Capacitor_SMD:C_0402_1005Metric" H 2188 3000 50  0001 C CNN
 F 3 "~" H 2150 3150 50  0001 C CNN
 	1    2150 3150
@@
 F 0 "C12" V 2000 3650 50  0000 C CNN
 F 1 "12pF" V 2300 3650 50  0000 C CNN
-F 2 "" H 2188 3500 50  0001 C CNN
+F 2 "Capacitor_SMD:C_0402_1005Metric" H 2188 3500 50  0001 C CNN
 F 3 "~" H 2150 3650 50  0001 C CNN
 	1    2150 3650
@@
 F 0 "L1" V 8850 3900 50  0000 C CNN
 F 1 "3.9nH" V 8700 3900 50  0000 C CNN
-F 2 "" H 8750 3900 50  0001 C CNN
+F 2 "Inductor_SMD:L_0402_1005Metric" H 8750 3900 50  0001 C CNN
 F 3 "~" H 8750 3900 50  0001 C CNN
 	1    8750 3900
@@
 F 0 "L2" H 5252 1896 50  0000 L CNN
 F 1 "10µH" H 5252 1805 50  0000 L CNN
-F 2 "" H 5200 1850 50  0001 C CNN
+F 2 "Inductor_SMD:L_0603_1608Metric" H 5200 1850 50  0001 C CNN
 F 3 "~" H 5200 1850 50  0001 C CNN
 	1    5200 1850
@@
 F 0 "L3" H 5253 1496 50  0000 L CNN
 F 1 "15nH" H 5253 1405 50  0000 L CNN
-F 2 "" H 5200 1450 50  0001 C CNN
+F 2 "Inductor_SMD:L_0402_1005Metric" H 5200 1450 50  0001 C CNN
 F 3 "~" H 5200 1450 50  0001 C CNN
 	1    5200 1450
@@
 F 0 "X1" V 8550 2600 50  0000 C CNN
 F 1 "32MHz" V 8750 2650 50  0000 C CNN
-F 2 "" H 8650 2450 50  0001 C CNN
+F 2 "Crystal:Crystal_SMD_2016-4Pin_2.0x1.6mm" H 8650 2450 50  0001 C CNN
 F 3 "~" H 8650 2450 50  0001 C CNN
 	1    8650 2450
@@
 F 0 "X2" V 2400 3550 50  0000 C CNN
 F 1 "32.768kHz" V 2600 3700 50  0000 C CNN
-F 2 "" H 2500 3400 50  0001 C CNN
+F 2 "Crystal:Crystal_SMD_3215-2Pin_3.2x1.5mm" H 2500 3400 50  0001 C CNN
 F 3 "~" H 2500 3400 50  0001 C CNN
 	1    2500 3400
@@
 F 0 "U1" H 7000 2700 50  0000 L CNN
 F 1 "nRF52832-QFAA" H 7000 2600 50  0000 L CNN
-F 2 "" H 5250 3650 50  0001 C CNN
+F 2 "Package_DFN_QFN:QFN-48-1EP_6x6mm_P0.4mm_EP4.2x4.2mm" H 5250 3650 50  0001 C CNN
 F 3 "" H 5250 3650 50  0001 C CNN
 	1    5900 3850
@@
 F 0 "C8" H 7915 2896 50  0000 L CNN
 F 1 "100nF" H 7915 2805 50  0000 L CNN
-F 2 "" H 7838 2700 50  0001 C CNN
+F 2 "Capacitor_SMD:C_0402_1005Metric" H 7838 2700 50  0001 C CNN
 F 3 "~" H 7800 2850 50  0001 C CNN
 	1    7800 2850
@@
 $EndComp
 Connection ~ 5850 1600
+$Comp
+L power:PWR_FLAG #FLG0102
+U 1 1 5CFC40F1
+P 9600 2700
+F 0 "#FLG0102" H 9600 2775 50  0001 C CNN
+F 1 "PWR_FLAG" V 9600 2828 50  0000 L CNN
+F 2 "" H 9600 2700 50  0001 C CNN
+F 3 "~" H 9600 2700 50  0001 C CNN
+	1    9600 2700
+	0    1    1    0
+$EndComp
 $EndSCHEMATC
