File: nRF52832.kicad_pcb (KiCad board)
At the start: 2 copper layers, 20.4 x 16 mm, 18 parts, among them U1 nRF52832-QFAA, X1 32MHz, X2 32.768kHz

Commit message: Adding RF track
Routing:
- net /RF: track 0.00 -> 1.33 mm
Other:
- net class RF added: clearance 0.1, trace_width 0.45, via_dia 0.8, via_drill 0.4
Changed lines of the file:
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@@
     (thickness 1.6)
     (drawings 8)
-    (tracks 232)
+    (tracks 233)
     (zones 0)
     (modules 18)
@@
     (add_net /P0.30-AIN6)
     (add_net /P0.31-AIN7)
-    (add_net /RF)
     (add_net /SWDCLK)
     (add_net /SWDIO)
@@
     (uvia_drill 0.1)
     (add_net VDD)
+  )
+  (net_class RF ""
+    (clearance 0.1)
+    (trace_width 0.45)
+    (via_dia 0.8)
+    (via_drill 0.4)
+    (uvia_dia 0.3)
+    (uvia_drill 0.1)
+    (add_net /RF)
   )
   (module Crystal:Crystal_SMD_3215-2Pin_3.2x1.5mm (layer F.Cu)
@@
   (gr_line (start 121.25 90.8) (end 121.25 77.25) (layer Edge.Cuts) (width 0.05))
   (gr_line (start 120.05 92) (end 102.1 92) (layer Edge.Cuts) (width 0.05))
-  (segment (start 109 91.7) (end 109 89.05) (width 0.25) (layer F.Cu) (net 38))
   (segment (start 115.3 84.1) (end 115.25 84.15) (width 0.25) (layer F.Cu) (net 1))
   (segment (start 115.25 84.15) (end 115.1 84.3) (width 0.25) (layer F.Cu) (net 1))
@@
   (segment (start 101.63 86.72) (end 102.35 86) (width 0.25) (layer F.Cu) (net 11))
   (segment (start 101.63 88.2) (end 101.63 86.72) (width 0.25) (layer F.Cu) (net 11))
+  (segment (start 119.52 87.15) (end 120.85 87.15) (width 0.45) (layer F.Cu) (net 12))
   (segment (start 107.6 80.975) (end 108.375 81.75) (width 0.25) (layer F.Cu) (net 13))
   (segment (start 108.8 81.75) (end 108.94999 81.89999) (width 0.25) (layer F.Cu) (net 13))
@@
   (segment (start 109.8 88.7) (end 109.8 91.7) (width 0.25) (layer F.Cu) (net 36))
   (segment (start 109.4 88.7) (end 109.4 91.7) (width 0.25) (layer F.Cu) (net 37))
+  (segment (start 109 91.7) (end 109 89.05) (width 0.25) (layer F.Cu) (net 38))
   (segment (start 106.6 88.7) (end 106.6 91.7) (width 0.25) (layer F.Cu) (net 39))
   (segment (start 106.6 88.7) (end 106.6 88.45) (width 0.25) (layer F.Cu) (net 39))
